Commit message: completed A.002

File: nuturtle_description/urdf/diff_drive.urdf.xacro (robot description, xacro)
@@ -11,4 +11,5 @@
 <xacro:property name="r" value="${params['wheel_radius']}" />
 <xacro:property name="h" value="${params['wheel_width']}" />
+<xacro:property name="r_bc" value="${(r - H/2)/2}" />
 <!-- <xacro:property name="m" value="${params['m']}" /> -->
   <!-- Include Macros -->
@@ -24,5 +25,5 @@
   <r_box name="base_link"
               origin_rpy="0 0 0" origin_xyz="0 0 0"
-              size="${L} ${W} ${H}"
+              size="${L} ${W - h} ${H}"
               matname="red_mat"
               rgba="1 0 0 1"/>
@@ -57,7 +58,7 @@
   <r_sph name="ball_caster"
               origin_rpy="0 0 0" origin_xyz="0 0 0"
-              radius="${r/4}"
-              matname="black_mat"
-              rgba="0 0 0 1"/>
+              radius="${r_bc}"
+              matname="green_mat"
+              rgba="0 1 0 1"/>
   <!-- Joints -->
   <frame_joint name="basefootprint_base" type="fixed"
@@ -67,5 +68,5 @@
   <wheel_joint name="right_wheel_axle" type="continuous"
                     axis_xyz="0 1 0"
-                    origin_rpy="0 0 0" origin_xyz="${r-L/2} -${W-h} 0"
+                    origin_rpy="0 0 0" origin_xyz="${r-L/2} -${W/2} 0"
                     parent="base_link" child="rr_wheel"
                     effort="100"
@@ -76,5 +77,5 @@
   <wheel_joint name="left_wheel_axle" type="continuous"
                     axis_xyz="0 1 0"
-                    origin_rpy="0 0 0" origin_xyz="${r-L/2} ${W-h} 0"
+                    origin_rpy="0 0 0" origin_xyz="${r-L/2} ${W/2} 0"
                     parent="base_link" child="rl_wheel"
                     effort="100"
@@ -94,5 +95,5 @@
   <wheel_joint name="base_bc" type="fixed"
                     axis_xyz="1 1 1"
-                    origin_rpy="0 0 0" origin_xyz="${L/2 - r/2} 0 -${H - r/4}"
+                    origin_rpy="0 0 0" origin_xyz="${L/2 - r_bc} 0 -${H/2 + r_bc}"
                     parent="base_link" child="ball_caster"
                     effort="0"

Commit message: tried to modify xacro, still teleports...

File: nuturtle_description/urdf/diff_drive.urdf.xacro (robot description, xacro)
@@ -21,5 +21,5 @@
   <!-- Robot description -->
   <!-- Links -->
-  <link name="base_footprint"/>
+  <!-- <link name="base_footprint"/> -->
   <!-- Base Link -->
   <r_box name="base_link"
@@ -62,7 +62,7 @@
               rgba="0 1 0 0.8"/>
   <!-- Joints -->
-  <frame_joint name="basefootprint_base" type="fixed"
+<!--   <frame_joint name="basefootprint_base" type="fixed"
                     origin_rpy="0 0 0" origin_xyz="0 0 ${r}"
-                    parent="base_footprint" child="base_link"/>
+                    parent="base_footprint" child="base_link"/> -->
   <!-- Joint 1: Base - RR Wheel -->
   <wheel_joint name="right_wheel_axle" type="continuous"

Commit message: re-added base_footprint so robot rides above plane. Still works the same

File: nuturtle_description/urdf/diff_drive.urdf.xacro (robot description, xacro)
@@ -21,5 +21,5 @@
   <!-- Robot description -->
   <!-- Links -->
-  <!-- <link name="base_footprint"/> -->
+  <link name="base_footprint"/>
   <!-- Base Link -->
   <r_box name="base_link"
@@ -62,7 +62,7 @@
               rgba="0 1 0 0.8"/>
   <!-- Joints -->
-<!--   <frame_joint name="basefootprint_base" type="fixed"
+  <frame_joint name="basefootprint_base" type="fixed"
                     origin_rpy="0 0 0" origin_xyz="0 0 ${r}"
-                    parent="base_footprint" child="base_link"/> -->
+                    parent="base_footprint" child="base_link"/>
   <!-- Joint 1: Base - RR Wheel -->
   <wheel_joint name="right_wheel_axle" type="continuous"

Commit message: modified xacro to look like actual turtlebot (will mount lidar later)

File: nuturtle_description/urdf/diff_drive.urdf.xacro (robot description, xacro)
@@ -8,8 +8,9 @@
 <xacro:property name="W" value="${params['wheel_base']}" />
 <xacro:property name="H" value="${params['chassis_thickness']}" />
+<xacro:property name="w_off" value="${params['wheel_axle_offset']}" />
 <!-- <xacro:property name="M" value="${params['M']}" /> -->
 <xacro:property name="r" value="${params['wheel_radius']}" />
 <xacro:property name="h" value="${params['wheel_width']}" />
-<xacro:property name="r_bc" value="${(r - H/2)/2}" />
+<xacro:property name="r_bc" value="${(r - w_off)/2}" />
 <!-- <xacro:property name="m" value="${params['m']}" /> -->
   <!-- Include Macros -->
@@ -63,10 +64,10 @@
   <!-- Joints -->
   <xacro:frame_joint name="basefootprint_base" type="fixed"
-                    origin_rpy="0 0 0" origin_xyz="0 0 ${r}"
+                    origin_rpy="0 0 0" origin_xyz="0 0 ${H/2 + r - w_off}"
                     parent="base_footprint" child="base_link"/>
   <!-- Joint 1: Base - RR Wheel -->
   <xacro:wheel_joint name="right_wheel_axle" type="continuous"
                     axis_xyz="0 1 0"
-                    origin_rpy="0 0 0" origin_xyz="0 -${W/2} 0"
+                    origin_rpy="0 0 0" origin_xyz="0 -${W/2} -${H/2 - w_off}"
                     parent="base_link" child="rr_wheel"
                     effort="100"
@@ -77,5 +78,5 @@
   <xacro:wheel_joint name="left_wheel_axle" type="continuous"
                     axis_xyz="0 1 0"
-                    origin_rpy="0 0 0" origin_xyz="0 ${W/2} 0"
+                    origin_rpy="0 0 0" origin_xyz="0 ${W/2} -${H/2 - w_off}"
                     parent="base_link" child="rl_wheel"
                     effort="100"

Commit message: added inertia and reversed turtlebot direction to match real

File: nuturtle_description/urdf/diff_drive.urdf.xacro (robot description, xacro)
@@ -14,4 +14,6 @@
 <xacro:property name="r_bc" value="${(r - w_off)/2}" />
 <!-- <xacro:property name="m" value="${params['m']}" /> -->
+<xacro:property name="m_c" value="${params['chassis_mass']}" />
+<xacro:property name="m_w" value="${params['wheel_mass']}" />
   <!-- Include Macros -->
   <xacro:include filename="$(find nuturtle_description)/urdf/diff_drive_macro.xacro" />
@@ -25,8 +27,12 @@
   <!-- Base Link -->
   <xacro:r_box name="base_link"
-              origin_rpy="0 0 0" origin_xyz="${L/2 - r} 0 0"
+              origin_rpy="0 0 0" origin_xyz="-${L/2 - r} 0 0"
               size="${L} ${W - h} ${H}"
               matname="red_mat"
-              rgba="1 0 0 0.8"/>
+              rgba="1 0 0 0.8"
+              mass="${m_c}"
+              ixx="${m_c * ( (H*H) + ((W-h)*(W-h)) ) / 12.0}" ixy="0" ixz="0"
+              iyy="${m_c * ( (L*L) + ((W-h)*(W-h)) ) / 12.0}" iyz="0"
+              izz="${m_c * ((H*H) + (L*L)) / 12.0}"/>
   <!-- Rear Right Wheel -->
   <xacro:r_cyl name="rr_wheel"
@@ -35,5 +41,9 @@
               radius="${r}"
               matname="black_mat"
-              rgba="0 0 0 0.8"/>
+              rgba="0 0 0 0.8"
+              mass="0.1"
+              ixx="${0.5 * m_w * (r*r)}" ixy="0" ixz="0"
+              iyy="${m_w * ((3*r*r)+ (L*L)) / 12.0}" iyz="0"
+              izz="${m_w * ((3*r*r)+ (L*L)) / 12.0}"/>
   <!-- Rear Left Wheel -->
   <xacro:r_cyl name="rl_wheel"
@@ -42,5 +52,9 @@
               radius="${r}"
               matname="black_mat"
-              rgba="0 0 0 0.8"/>
+              rgba="0 0 0 0.8"
+              mass="0.1"
+              ixx="${0.5 * m_w * (r*r)}" ixy="0" ixz="0"
+              iyy="${m_w * ((3*r*r)+ (L*L)) / 12.0}" iyz="0"
+              izz="${m_w * ((3*r*r)+ (L*L)) / 12.0}"/>
   <!-- Top Caster Wheel -->
   <!-- <r_sph name="tc_wheel"
@@ -62,4 +76,6 @@
               matname="green_mat"
               rgba="0 1 0 0.8"/>
+  <!-- Scanner -->
+  <link name="base_scan"/>
   <!-- Joints -->
   <xacro:frame_joint name="basefootprint_base" type="fixed"
@@ -96,5 +112,5 @@
   <xacro:wheel_joint name="base_bc" type="fixed"
                     axis_xyz="1 1 1"
-                    origin_rpy="0 0 0" origin_xyz="${L/2 + r - r_bc} 0 -${H/2 + r_bc}"
+                    origin_rpy="0 0 0" origin_xyz="-${L/2 + r - r_bc} 0 -${H/2 + r_bc}"
                     parent="base_link" child="ball_caster"
                     effort="0"
@@ -102,3 +118,6 @@
                     damping="0"
                     friction="0"/>
+  <xacro:frame_joint name="base_scan" type="fixed"
+                    origin_rpy="0 0 0" origin_xyz="0 0 ${H/2}"
+                    parent="base_link" child="base_scan"/>
 </robot>

File: nuturtle_description/urdf/diff_drive_macro.xacro (robot description, xacro)
@@ -18,5 +18,5 @@
     </joint>
   </xacro:macro>
-  <xacro:macro name="r_box" params="name origin_xyz origin_rpy size matname rgba">
+  <xacro:macro name="r_box" params="name origin_xyz origin_rpy size mass ixx ixy ixz iyy iyz izz matname rgba">
     <link name="${name}">
       <visual>
@@ -29,5 +29,5 @@
         </material>
       </visual>
-      <!-- <collision>
+      <collision>
         <origin rpy="${origin_rpy}" xyz="${origin_xyz}" />
         <geometry>
@@ -41,8 +41,8 @@
                  iyy="${iyy}" iyz="${iyz}"
                  izz="${izz}" />
-      </inertial> -->
+      </inertial>
     </link>
   </xacro:macro>
-  <xacro:macro name="r_cyl" params="name origin_xyz origin_rpy length radius matname rgba">
+  <xacro:macro name="r_cyl" params="name origin_xyz origin_rpy length radius mass ixx ixy ixz iyy iyz izz matname rgba">
     <link name="${name}">
       <visual>
@@ -55,5 +55,5 @@
         </material>
       </visual>
-      <!-- <collision>
+      <collision>
         <origin rpy="${origin_rpy}" xyz="${origin_xyz}" />
         <geometry>
@@ -67,5 +67,5 @@
                  iyy="${iyy}" iyz="${iyz}"
                  izz="${izz}" />
-      </inertial> -->
+      </inertial>
     </link>
   </xacro:macro>
@@ -81,5 +81,5 @@
         </material>
       </visual>
-      <!-- <collision>
+      <collision>
         <origin rpy="${origin_rpy}" xyz="${origin_xyz}" />
         <geometry>
@@ -87,5 +87,5 @@
         </geometry>
       </collision>
-      <inertial>
+      <!-- <inertial>
         <origin rpy="${origin_rpy}" xyz="${origin_xyz}" />
         <mass value="${mass}"/>

Commit message: completed G.004 and G.005 (fixed launchfile world arg)

File: nuturtle_description/urdf/diff_drive.urdf.xacro (robot description, xacro)
@@ -119,5 +119,5 @@
                     friction="0"/>
   <xacro:frame_joint name="base_scan" type="fixed"
-                    origin_rpy="0 0 0" origin_xyz="0 0 ${H/2}"
-                    parent="base_link" child="base_scan"/>
+                    origin_rpy="0 0 0" origin_xyz="0 0 ${H/2 + r_bc}"
+                    parent="base_link" child="base_scan"/> <!-- Add small offset to laser scanner -->
 </robot>

File: nuturtle_gazebo/urdf/diff_drive.gazebo.xacro (robot description, xacro)
@@ -61,3 +61,36 @@
     <!-- <fdir1>1 1 0</fdir1> --> <!-- friction direction -->
 </gazebo>
+<!-- Laser Scanner -->
+<gazebo reference="base_scan">
+  <material>Gazebo/Orange</material>
+  <sensor type="ray" name="lds_lfcd_sensor">
+    <pose>0 0 0 0 0 0</pose>
+    <visualize>true</visualize>
+    <update_rate>5</update_rate>
+    <ray>
+      <scan>
+        <horizontal>
+          <samples>360</samples>
+          <resolution>1</resolution>
+          <min_angle>0.0</min_angle>
+          <max_angle>6.28319</max_angle>
+        </horizontal>
+      </scan>
+      <range>
+        <min>0.120</min>
+        <max>3.5</max>
+        <resolution>0.015</resolution>
+      </range>
+      <noise>
+        <type>gaussian</type>
+        <mean>0.0</mean>
+        <stddev>0.01</stddev>
+      </noise>
+    </ray>
+    <plugin name="gazebo_ros_lds_lfcd_controller" filename="libgazebo_ros_laser.so">
+      <topicName>scan</topicName>
+      <frameName>base_scan</frameName>
+    </plugin>
+  </sensor>
+</gazebo>
 </robot>
